File: amp-board/amp-board.kicad_pcb (KiCad board)
At the start: 4 copper layers, 27 parts, among them J1 COIL, J2 Vin, J3 GND, J4 Vin, J5 Vin, Q1 2N3904, Q2 IRF9610, U1 MCP1703T-5002E, U3 NE5534

Commit message: step2 layout
Parts:
- removed J5: Vin, Connector_PinSocket_2.54mm:PinSocket_1x01_P2.54mm_Vertical
- added C11: 100u, Capacitor_Tantalum_SMD:CP_EIA-7361-438_AVX-U_Pad2.18x3.30mm_HandSolder, B.Cu at (120.1, 99.2)
- added C12: 100u, Capacitor_Tantalum_SMD:CP_EIA-7361-438_AVX-U_Pad2.18x3.30mm_HandSolder, B.Cu at (120.1, 106.0)
- added C3: 100u, Capacitor_Tantalum_SMD:CP_EIA-7361-438_AVX-U_Pad2.18x3.30mm_HandSolder, B.Cu at (140.5, 96.4)
- added C5: 22u, Capacitor_SMD:C_1206_3216Metric, B.Cu at (130.0, 106.0)
- added C6: 22u, Capacitor_SMD:C_1206_3216Metric, B.Cu at (130.0, 109.1)
- added C7: 100u, Capacitor_Tantalum_SMD:CP_EIA-7361-438_AVX-U_Pad2.18x3.30mm_HandSolder, B.Cu at (120.1, 85.6)
- added C8: 100u, Capacitor_Tantalum_SMD:CP_EIA-7361-438_AVX-U_Pad2.18x3.30mm_HandSolder, B.Cu at (120.1, 92.4)
- added Q3: 2N3904, Package_TO_SOT_SMD:SOT-23, B.Cu at (136.0, 85.2)
- added R3: 10k, Resistor_SMD:R_0805_2012Metric, B.Cu at (139.6, 83.1)
- added R9: 20k, Resistor_SMD:R_0805_2012Metric, B.Cu at (131.3, 85.0)
- added U2: LT1054, Package_DIP:DIP-8_W8.89mm_SMDSocket_LongPads, B.Cu at (131.3, 97.9)
- J2: value Vin -> BAT+; footprint Connector_PinSocket_2.54mm:PinSocket_1x01_P2.54mm_Vertical -> Connector_Wire:SolderWirePad_1x01_SMD_2x4mm
- J3: value GND -> BAT-; footprint Connector_PinSocket_2.54mm:PinSocket_1x01_P2.54mm_Vertical -> Connector_Wire:SolderWirePad_1x01_SMD_2x4mm
- J4: value Vin -> PWM; footprint Connector_PinSocket_2.54mm:PinSocket_1x01_P2.54mm_Vertical -> Connector_Wire:SolderWirePad_1x01_SMD_2x4mm
- moved RV1 47.4 mm to (46.7, 95.9), turned to 0 degrees
- moved R7 43.6 mm to (44.2, 92.6), turned to -90 degrees
- moved TP1 41.5 mm to (51.1, 92.2), turned to 0 degrees
- moved C9 36.0 mm to (49.6, 88.1), turned to 0 degrees
- moved U1 32.0 mm to (89.9, 50.3)
- moved C1 32.0 mm to (96.0, 47.8)
- moved C2 32.0 mm to (96.0, 52.8)
- moved R8 21.8 mm to (55.4, 78.0), turned to 90 degrees
- moved U3 21.5 mm to (48.3, 77.5), turned to -90 degrees
- moved R6 12.7 mm to (44.2, 68.6)
- moved C10 7.84 mm to (49.6, 68.6), turned to 180 degrees
- moved R5 6.32 mm to (49.8, 62.0)
- moved D1 4.83 mm to (45.5, 63.0), turned to 180 degrees
- moved D2 4.34 mm to (45.4, 65.6), turned to 0 degrees
- moved J3 3.05 mm to (81.8, 52.8)
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Routing:
- net BAT-: track 110.4 -> 248.9 mm
- net BAT+: track 23.6 -> 56.5 mm
- net V+: track 15.7 -> 35.3 mm, vias 0 -> 3
- net V-: track 13.0 -> 32.2 mm, vias 0 -> 1
- net Net-(Q3-Pad3): track 0.00 -> 10.7 mm
- net Net-(R9-Pad1): track 0.00 -> 8.16 mm
- net Net-(C5-Pad1): track 0.00 -> 7.96 mm
- net Net-(C5-Pad2): track 0.00 -> 7.88 mm
- net PWM: track 3.15 -> 7.63 mm, vias 0 -> 2
- net AMP_SIG: track 17.1 -> 20.0 mm
- net Net-(Q3-Pad1): track 0.00 -> 2.75 mm
- net Net-(D1-Pad2): track 18.6 -> 19.3 mm
- net Net-(R6-Pad2): track 16.8 -> 17.3 mm
Other:
- board outline added: 59.9 x 65 mm
- board text added: "BAT+"
- board text added: "BAT-"
- board text added: "G"
- board text added: "Metal detector board step 2 preamp positive PSU negative PSU"
- board text added: "RAW"
- board text added: "SIG"

Commit message: 2023-07-05
Parts:
- removed TP1, TP2: TestPoint, TestPoint:TestPoint_2Pads_Pitch2.54mm_Drill0.8mm
- added ?: , , F.Cu at (175.3, 116.8)
- added ?: , , F.Cu at (175.3, 67.3)
- added ?: , , F.Cu at (81.3, 67.3)
- added ?: , , F.Cu at (81.3, 116.8)
- added ?: , , F.Cu at (160.1, 91.4)
- added BZ1: Buzzer, !my-kicad-library:Buzzer-GT-0905A, F.Cu at (88.3, 95.9)
- added C13: 100n, Capacitor_SMD:C_1206_3216Metric, B.Cu at (139.4, 109.6)
- added C14: 100n, Capacitor_SMD:C_1206_3216Metric, B.Cu at (131.4, 101.0)
- added C15: 100n, Capacitor_SMD:C_1206_3216Metric, B.Cu at (118.5, 113.4)
- added C16: 470nF, Capacitor_SMD:C_1206_3216Metric, B.Cu at (126.6, 100.4)
- added C17: 100n, Capacitor_SMD:C_1206_3216Metric, B.Cu at (117.5, 101.0)
- added C18: 470nF, Capacitor_SMD:C_1206_3216Metric, B.Cu at (131.9, 108.5)
- added C19: 470nF, Capacitor_SMD:C_1206_3216Metric, B.Cu at (138.0, 101.0)
- added C20: 100nF, Capacitor_SMD:C_1206_3216Metric, B.Cu at (144.8, 104.8)
- added C21: 100n, Capacitor_SMD:C_1206_3216Metric, B.Cu at (150.7, 112.1)
- added C22: 470nF, Capacitor_SMD:C_1206_3216Metric, B.Cu at (114.3, 88.9)
- added D3: 1N4148, Diode_SMD:D_1206_3216Metric, B.Cu at (102.2, 109.7)
- added J5: AudioJack3, !my-kicad-library:audio-jack, F.Cu at (88.3, 114.8)
- added Q4: MMBTA13LT3G, Package_TO_SOT_SMD:SOT-23, B.Cu at (105.4, 109.7)
- added Q5: 2N3906_2A, Package_TO_SOT_SMD:SOT-23, B.Cu at (109.2, 102.9)
- added Q6: 2N3906_2A, Package_TO_SOT_SMD:SOT-23, B.Cu at (125.5, 110.5)
- added Q7: 2N3906_2A, Package_TO_SOT_SMD:SOT-23, B.Cu at (105.4, 102.9)
- added R10: 1k, Resistor_SMD:R_0805_2012Metric, B.Cu at (125.7, 106.3)
- added R11: 1k, Resistor_SMD:R_0805_2012Metric, B.Cu at (125.7, 104.3)
- added R12: 220k, Resistor_SMD:R_0805_2012Metric, B.Cu at (128.7, 100.5)
- added R13: 220k, Resistor_SMD:R_0805_2012Metric, B.Cu at (129.3, 108.0)
- added R14: 220k, Resistor_SMD:R_0805_2012Metric, B.Cu at (138.9, 98.6)
- added R15: 1k, Resistor_SMD:R_0805_2012Metric, B.Cu at (93.8, 115.2)
- added R16: 100k, Resistor_SMD:R_0805_2012Metric, B.Cu at (142.6, 105.3)
- added R17: 47k, Resistor_SMD:R_0805_2012Metric, B.Cu at (99.7, 107.0)
- added R18: 22k, Resistor_SMD:R_0805_2012Metric, B.Cu at (93.7, 112.6)
- added R19: 22k, Resistor_SMD:R_0805_2012Metric, B.Cu at (144.8, 109.0)
- added R20: 100k, Resistor_SMD:R_0805_2012Metric, B.Cu at (110.8, 109.7)
- added R21: 150, Resistor_SMD:R_0805_2012Metric, B.Cu at (108.6, 109.7)
- added R22: 10k, Resistor_SMD:R_0805_2012Metric, B.Cu at (112.0, 102.9)
- added R23: 10k, Resistor_SMD:R_0805_2012Metric, B.Cu at (122.7, 110.5)
- added R24: 10k, Resistor_SMD:R_0805_2012Metric, B.Cu at (102.6, 102.9)
- added R25: 10k, Resistor_SMD:R_0805_2012Metric, B.Cu at (151.8, 100.3)
- added R26: 10k, Resistor_SMD:R_0805_2012Metric, B.Cu at (150.4, 105.2)
- added R27: 10k, Resistor_SMD:R_0805_2012Metric, B.Cu at (164.4, 106.2)
- added R28: 1k, Resistor_SMD:R_0805_2012Metric, B.Cu at (118.7, 98.4)
- added REF**: SolderWirePad_1x01_SMD_2x4mm, Connector_Wire:SolderWirePad_1x01_SMD_2x4mm, B.Cu at (149.4, 107.8)
- added RV_THRESHOLD1: 10k, Connector_JST:JST_EH_B3B-EH-A_1x03_P2.50mm_Vertical, F.Cu at (97.8, 110.1)
- added RV_TIMING1: 10k, Connector_JST:JST_EH_B3B-EH-A_1x03_P2.50mm_Vertical, F.Cu at (156.1, 114.5)
- added RV_VOLUME1: 1k, Connector_JST:JST_EH_B3B-EH-A_1x03_P2.50mm_Vertical, F.Cu at (97.8, 98.5)
- added SW1: SW_SPDT, Connector_JST:JST_EH_B3B-EH-A_1x03_P2.50mm_Vertical, F.Cu at (97.8, 87.2)
- added U4: LM358, Package_SO:SOIC-8_3.9x4.9mm_P1.27mm, B.Cu at (137.5, 105.4)
- added U5: 4066, Package_SO:SO-14_3.9x8.65mm_P1.27mm, B.Cu at (117.4, 107.3)
- added U6: ATtiny85-20P, Package_DIP:DIP-8_W7.62mm, F.Cu at (161.6, 110.3)
- D1, D2: footprint !my-kicad-library:D_4148_SMD -> Diode_SMD:D_1206_3216Metric
- R4: value 3.3 2W -> 5.1 1W+; footprint Resistor_THT:R_Axial_DIN0614_L14.3mm_D5.7mm_P5.08mm_Vertical -> Resistor_THT:R_Axial_DIN0411_L9.9mm_D3.6mm_P12.70mm_Horizontal
- R_DAMP1: value 1k 0.75W+ -> 1k 0.25W+; footprint Resistor_THT:R_Axial_DIN0614_L14.3mm_D5.7mm_P5.08mm_Vertical -> Resistor_THT:R_Axial_DIN0207_L6.3mm_D2.5mm_P10.16mm_Horizontal
- U2: footprint Package_DIP:DIP-8_W8.89mm_SMDSocket_LongPads -> Package_SO:SOIC-8_3.9x4.9mm_P1.27mm
- moved J4 113.3 mm to (156.5, 78.7), turned to 180 degrees
- moved R1 110.6 mm to (156.6, 82.9), turned to -90 degrees
- moved Q1 108.4 mm to (153.5, 81.8)
- moved R2 100.1 mm to (153.5, 77.7), turned to 90 degrees
- moved R4 94.6 mm to (153.0, 70.6), turned to 180 degrees
- moved J1 93.8 mm to (135.3, 76.2), turned to 180 degrees
- moved Q2 93.8 mm to (145.4, 77.1)
- moved R_DAMP1 91.4 mm to (139.8, 83.8), turned to 180 degrees
- moved C4 91.4 mm to (160.0, 73.3)
- moved J2 86.4 mm to (163.4, 70.6)
- moved J3 86.4 mm to (161.6, 85.9)
- moved C1 83.1 mm to (174.1, 76.2)
- moved C2 83.1 mm to (174.1, 81.3)
- moved U1 83.1 mm to (168.0, 78.7)
- moved D1 82.8 mm to (126.3, 81.1), turned to 90 degrees
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- renumbered RV1 to RV_OPAMP1
Connections:
- net AMP_SIG renamed Net-(R8-Pad1)
- net Net-(D1-Pad2) renamed /raw sig
Routing:
- net V+: track 35.3 -> 282.0 mm, vias 3 -> 4
- net BAT-: track 248.9 -> 468.5 mm, vias 4 -> 3
- net V-: track 32.2 -> 154.0 mm, vias 1 -> 5
- net THRESHOLD: track 0.00 -> 88.7 mm, vias 0 -> 2
- net PWM: track 7.63 -> 91.1 mm, vias 2 -> 3
- net BAT+: track 56.5 -> 138.5 mm
- net Net-(Q7-Pad1): track 0.00 -> 80.3 mm, vias 0 -> 2
- net Net-(Q5-Pad1): track 0.00 -> 54.5 mm, vias 0 -> 2
- net Net-(D3-Pad2): track 0.00 -> 52.8 mm
- net Net-(J5-PadR): track 0.00 -> 37.7 mm
- net Net-(Q6-Pad1): track 0.00 -> 27.6 mm, vias 0 -> 2
- net AMP_SIG: track 0.00 -> 24.2 mm
- net /collector: track 0.00 -> 18.1 mm, vias 0 -> 1
- net /drlng-base: track 0.00 -> 16.9 mm
- net AUDIO_PWM: track 0.00 -> 16.4 mm
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Other:
- board size 59.9 x 65 mm -> 100.6 x 56.1 mm
- board text added: "AMP SIG"
- board text added: "AUDIO"
- board text added: "AUDIO sw"
- board text added: "EFE"
- board text added: "MAIN"
- board text added: "Metal detector step 3"
- board text added: "RAW SIG"
- board text added: "out1"
- board text added: "out2"
- board text added: "threshold"
- board text added: "timing"
- board text added: "volume"
- board text removed: "G"
- board text removed: "Metal detector board step 2 preamp positive PSU negative PSU"
- board text removed: "RAW"
- board text removed: "SIG"
