File: amp-board/amp-board.kicad_sch (KiCad schematic)
At the start: 27 parts, among them J1 COIL, J2 Vin, J3 GND, J4 Vin, J5 Vin, Q1 2N3904, Q2 IRF9610, U1 MCP1703T-5002E, U3 NE5534

Commit message: step2 layout
Parts:
- removed J5: Vin, Connector_PinSocket_2.54mm:PinSocket_1x01_P2.54mm_Vertical, symbol Connector:Conn_01x01_Female
- added C11, C12, C3, C7, C8: 100u, Capacitor_Tantalum_SMD:CP_EIA-7361-438_AVX-U_Pad2.18x3.30mm_HandSolder, symbol Device:C_Polarized_US
- added C5, C6: 22u, Capacitor_SMD:C_1206_3216Metric, symbol Device:C
- added Q3: 2N3904, Package_TO_SOT_SMD:SOT-23, symbol !my-kicad-library:2N3904
- added R3: 10k, Resistor_SMD:R_0805_2012Metric, symbol Device:R_US
- added R9: 20k, Resistor_SMD:R_0805_2012Metric, symbol Device:R_US
- added U2: LT1054, Package_DIP:DIP-8_W8.89mm_SMDSocket_LongPads, symbol Regulator_SwitchedCapacitor:LT1054
- J2: value Vin -> BAT+; footprint Connector_PinSocket_2.54mm:PinSocket_1x01_P2.54mm_Vertical -> Connector_Wire:SolderWirePad_1x01_SMD_2x4mm
- J3: value GND -> BAT-; footprint Connector_PinSocket_2.54mm:PinSocket_1x01_P2.54mm_Vertical -> Connector_Wire:SolderWirePad_1x01_SMD_2x4mm
- J4: value Vin -> PWM; footprint Connector_PinSocket_2.54mm:PinSocket_1x01_P2.54mm_Vertical -> Connector_Wire:SolderWirePad_1x01_SMD_2x4mm
Connections:
- net GND: now also C11.1, C12.1, C3.2, C7.1, C8.1, Q3.2 (E), U2.3 (GND)
- net PWM: now also R3.1
- net V+: now also C3.1, U2.8 (V+)
- net V-: now also C11.2, C12.2, C7.2, C8.2, U2.5 (-VOUT)
- new net: Q3.1 (B), R3.2
- new net: Q3.3 (C), R9.2, U2.7 (OSC)
- new net: C5.1, C6.1, U2.2 (CAP+)
- new net: C5.2, C6.2, U2.4 (CAP-)
- new net: R9.1, U2.6 (VREF)
- no-connect marks 1 -> 2
Other:
- note added: "+5V"
- note added: "Keep away from signal path"
- note added: "Tantalum, low ESR"
- note added: "V+, 1KHz, 5%"
- note added: "ceramic"
- note added: "~ -4.65V ~ 2mA"

Commit message: 2023-07-05
Parts:
- removed TP1, TP2: TestPoint, TestPoint:TestPoint_2Pads_Pitch2.54mm_Drill0.8mm, symbol Connector:TestPoint
- added BZ1: Buzzer, !my-kicad-library:Buzzer-GT-0905A, symbol Device:Buzzer
- added C13, C14, C15, C17, C21: 100n, Capacitor_SMD:C_1206_3216Metric, symbol Device:C
- added C16, C18, C19, C22: 470nF, Capacitor_SMD:C_1206_3216Metric, symbol Device:C
- added C20: 100nF, Capacitor_SMD:C_1206_3216Metric, symbol Device:C
- added D3: 1N4148, Diode_SMD:D_1206_3216Metric, symbol Diode:1N4148
- added J5: AudioJack3, !my-kicad-library:audio-jack, symbol Connector:AudioJack3
- added Q4: MMBTA13LT3G, Package_TO_SOT_SMD:SOT-23, symbol Device:Q_NPN_Darlington_BEC
- added Q5, Q6, Q7: 2N3906_2A, Package_TO_SOT_SMD:SOT-23, symbol !my-kicad-library:2N3906_2A
- added R10, R11, R15, R28: 1k, Resistor_SMD:R_0805_2012Metric, symbol Device:R_US
- added R12, R13, R14: 220k, Resistor_SMD:R_0805_2012Metric, symbol Device:R_US
- added R16, R20: 100k, Resistor_SMD:R_0805_2012Metric, symbol Device:R_US
- added R17: 47k, Resistor_SMD:R_0805_2012Metric, symbol Device:R_US
- added R18, R19: 22k, Resistor_SMD:R_0805_2012Metric, symbol Device:R_US
- added R21: 150, Resistor_SMD:R_0805_2012Metric, symbol Device:R_US
- added R22, R23, R24, R25, R26, R27: 10k, Resistor_SMD:R_0805_2012Metric, symbol Device:R_US
- added RV_THRESHOLD1, RV_TIMING1: 10k, Connector_JST:JST_EH_B3B-EH-A_1x03_P2.50mm_Vertical, symbol Device:R_Potentiometer_US
- added RV_VOLUME1: 1k, Connector_JST:JST_EH_B3B-EH-A_1x03_P2.50mm_Vertical, symbol Device:R_Potentiometer_US
- added SW1: SW_SPDT, Connector_JST:JST_EH_B3B-EH-A_1x03_P2.50mm_Vertical, symbol Switch:SW_SPDT
- added U4: LM358, Package_SO:SOIC-8_3.9x4.9mm_P1.27mm, symbol Amplifier_Operational:LM358
- added U5: 4066, Package_SO:SO-14_3.9x8.65mm_P1.27mm, symbol 4xxx:4066
- added U6: ATtiny85-20P, Package_DIP:DIP-8_W7.62mm, symbol MCU_Microchip_ATtiny:ATtiny85-20P
- D1, D2: footprint !my-kicad-library:D_4148_SMD -> Diode_SMD:D_1206_3216Metric
- R4: value 3.3 2W -> 5.1 1W+; footprint Resistor_THT:R_Axial_DIN0614_L14.3mm_D5.7mm_P5.08mm_Vertical -> Resistor_THT:R_Axial_DIN0411_L9.9mm_D3.6mm_P12.70mm_Horizontal
- R_DAMP1: value 1k 0.75W+ -> 1k 0.25W+; footprint Resistor_THT:R_Axial_DIN0614_L14.3mm_D5.7mm_P5.08mm_Vertical -> Resistor_THT:R_Axial_DIN0207_L6.3mm_D2.5mm_P10.16mm_Horizontal
- U2: footprint Package_DIP:DIP-8_W8.89mm_SMDSocket_LongPads -> Package_SO:SOIC-8_3.9x4.9mm_P1.27mm
- renumbered RV1 to RV_OPAMP1
Connections:
- net AMP_SIG: now also C22.2, R28.2, U5.1, U5.3; no longer R8.1, U3.6
- net BAT+: now also RV_VOLUME1.1, SW1.2 (B)
- net GND: now also C13.2, C14.2, C15.2, C16.1, C17.2, C21.2, R12.2, R14.1, R15.1, R20.2, R21.2, R28.1, RV_THRESHOLD1.3, RV_TIMING1.3, U5.10, U5.6, U5.8, U5.9, U6.4 (GND)
- net PWM: now also U6.7 (PB2)
- net V+: now also C13.1, C17.1, C21.1, Q5.2 (E), Q6.2 (E), Q7.2 (E), RV_TIMING1.1, U4.8 (V+), U5.14 (VDD), U6.8 (VCC)
- net V-: now also C14.1, C15.1, R17.2, R22.2, R23.2, R24.2, U4.4 (V-), U5.7 (VSS)
- net raw sig: now reaches D1.2 (A), D2.1 (K), R5.1, U3.3 (+)
- new net: R18.2, RV_THRESHOLD1.2
- new net: C18.1, R10.1, R13.2, U4.2 (-)
- new net: Q7.1 (B), R27.2
- new net: Q5.1 (B), R25.2
- new net: D3.2 (A), R19.1
- new net: BZ1.1 (-), SW1.3 (C)
- new net: BZ1.2 (+), J5.T, RV_VOLUME1.2
- new net: R17.1, RV_THRESHOLD1.1
- new net: J5.R, SW1.1 (A)
- new net: C16.2, R11.1, R12.1, U4.3 (+)
- new net: RV_TIMING1.2, U6.2 (XTAL1/PB3)
- new net: C22.1, R8.1, U3.6
- new net: C19.2, R14.2, U4.5 (+)
- new net: Q6.1 (B), R26.2
- new net AUDIO_PIN: R27.1, U6.3 (XTAL2/PB4)
- new net AUDIO_PWM: Q7.3 (C), R24.1, U5.12
- new net EFE_SAMP: Q5.3 (C), R22.1, U5.5
- new net EFE_SAMP_PIN: R25.1, U6.5 (AREF/PB0)
- new net MAIN_SAMP: Q6.3 (C), R23.1, U5.13
- new net MAIN_SAMP_PIN: R26.1, U6.6 (PB1)
- new net RESULT_OUT: C20.2, R16.1, R19.2, U4.7
- new net THRESHOLD: C20.1, R15.2, R16.2, R18.1, U4.6 (-)
- new net collector: Q4.3 (C), RV_VOLUME1.3
- new net drlng-base: D3.1 (K), Q4.1 (B), R20.1, U5.11
- new net emitter: Q4.2 (E), R21.1
- new net out1: R10.2, U5.2
- new net out2: R11.2, U5.4
- new net stg1: C18.2, C19.1, R13.1, U4.1
- no-connect marks 2 -> 4
Other:
- moved on the sheet: C1, C2, U1
